File: Eink-Driver.kicad_pcb (KiCad board)
At the start: 2 copper layers, 21.6 x 32.7 mm, 46 parts, among them J3 Conn_01x24, Q1 AO3400A

Commit message: update
Parts:
- removed J3: Conn_01x24, Connector_FFC-FPC:Hirose_FH12-24S-0.5SH_1x24-1MP_P0.50mm_Horizontal
- removed kibuzzard-69635A03: G***, kibuzzard-69635A03
- added J1: Conn_01x24, Connector_FFC-FPC:Amphenol_F32Q-1A7x1-11024_1x24-1MP_P0.5mm_Horizontal, F.Cu at (135.9, 37.8)
- added kibuzzard-6A03540B: G***, kibuzzard-6A03540B, F.Cu at (135.9, 37.8)
- moved kibuzzard-69635A23 0.98 mm to (140.3, 39.1)
Routing:
- net GND: vias 0 -> 4
Other:
- board size 21.6 x 32.7 mm -> 21.6 x 30.1 mm
