File: Eink-Driver.kicad_sch (KiCad schematic)
At the start: 23 parts, among them J3 Conn_01x24, Q1 AO3400A

Commit message: update
Parts:
- removed J3: Conn_01x24, Connector_FFC-FPC:Hirose_FH12-24S-0.5SH_1x24-1MP_P0.50mm_Horizontal, symbol Connector_Generic:Conn_01x24
- added J1: Conn_01x24, Connector_FFC-FPC:Amphenol_F32Q-1A7x1-11024_1x24-1MP_P0.5mm_Horizontal, symbol Connector_Generic:Conn_01x24
Connections:
- net +3.3V: now also J1.10 (Pin_10), J1.9 (Pin_9)
- net BUSY: now also J1.16 (Pin_16)
- net DC: now also J1.14 (Pin_14)
- net DISPCS: now also J1.13 (Pin_13)
- net GDR: now also J1.23 (Pin_23)
- net GND: now also J1.17 (Pin_17), J1.8 (Pin_8)
- net MOSI: now also J1.11 (Pin_11)
- net RESE: now also J1.22 (Pin_22)
- net RESET: now also J1.15 (Pin_15)
- net SCLK: now also J1.12 (Pin_12)
- net TSCL: now also J1.19 (Pin_19)
- net TSDA: now also J1.18 (Pin_18)
- net VGH: now also J1.4 (Pin_4)
- net VGL: now also J1.2 (Pin_2)
- net at C22.2: now also J1.5 (Pin_5)
- net at C7.2: now also J1.6 (Pin_6)
- net at C16.2: now also J1.20 (Pin_20)
- net at C24.2: now also J1.1 (Pin_1)
- net at C2.2: now also J1.7 (Pin_7)
- net at C23.2: now also J1.3 (Pin_3)
- net at C6.2: now also J1.21 (Pin_21)
Changed lines of the file:
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@@
+	)
+	(symbol
+		(lib_id "Connector_Generic:Conn_01x24")
+		(at 241.3 71.12 0)
+		(mirror x)
+		(unit 1)
+		(exclude_from_sim no)
+		(in_bom yes)
+		(on_board yes)
+		(dnp no)
+		(property "Reference" "J1"
+			(at 243.84 71.1201 0)
+			(effects
+				(font
+					(size 1.27 1.27)
+				)
+				(justify left)
+			)
+		)
+		(property "Value" "Conn_01x24"
+			(at 243.84 68.5801 0)
+			(effects
+				(font
+					(size 1.27 1.27)
+				)
+				(justify left)
+			)
+		)
+		(property "Footprint" "Connector_FFC-FPC:Amphenol_F32Q-1A7x1-11024_1x24-1MP_P0.5mm_Horizontal"
+			(at 241.3 71.12 0)
+			(effects
+				(font
+					(size 1.27 1.27)
+				)
+				(hide yes)
+			)
+		)
+		(property "Datasheet" "~"
+			(at 241.3 71.12 0)
+			(effects
+				(font
+					(size 1.27 1.27)
+				)
+				(hide yes)
+			)
+		)
+		(property "Description" "Generic connector, single row, 01x24, script generated (kicad-library-utils/schlib/autogen/connector/)"
+			(at 241.3 71.12 0)
+			(effects
+				(font
+					(size 1.27 1.27)
+				)
+				(hide yes)
+			)
+		)
+		(pin "14"
+		)
+		(pin "9"
+		)
+		(pin "13"
+		)
+		(pin "20"
+		)
+		(pin "1"
+		)
+		(pin "23"
+		)
+		(pin "3"
+		)
+		(pin "4"
+		)
+		(pin "10"
+		)
+		(pin "11"
+		)
+		(pin "8"
+		)
+		(pin "5"
+		)
+		(pin "7"
+		)
+		(pin "6"
+		)
+		(pin "2"
+		)
+		(pin "12"
+		)
+		(pin "15"
+		)
+		(pin "16"
+		)
+		(pin "17"
+		)
+		(pin "18"
+		)
+		(pin "19"
+		)
+		(pin "21"
+		)
+		(pin "22"
+		)
+		(pin "24"
+		)
+		(instances
+			(project "Eink-Driver"
+				(path "/ff08cec3-484d-4cc6-8498-b7b3b5dcf0bf"
+					(reference "J1")
+					(unit 1)
+				)
+			)
+		)
 	)
 	(symbol
@@
 					(unit 1)
 				)
-			)
-		)
-	)
-	(symbol
-		(lib_id "Connector_Generic:Conn_01x24")
-		(at 241.3 71.12 0)
-		(mirror x)
-		(unit 1)
-		(exclude_from_sim no)
-		(in_bom yes)
-		(on_board yes)
-		(dnp no)
-		(property "Reference" "J3"
-			(at 243.84 71.1201 0)
-			(effects
-				(font
-					(size 1.27 1.27)
-				)
-				(justify left)
-			)
-		)
-		(property "Value" "Conn_01x24"
-			(at 243.84 68.5801 0)
-			(effects
-				(font
-					(size 1.27 1.27)
-				)
-				(justify left)
-			)
-		)
-		(property "Footprint" "Connector_FFC-FPC:Hirose_FH12-24S-0.5SH_1x24-1MP_P0.50mm_Horizontal"
-			(at 241.3 71.12 0)
-			(effects
-				(font
-					(size 1.27 1.27)
-				)
-				(hide yes)
-			)
-		)
-		(property "Datasheet" "~"
-			(at 241.3 71.12 0)
-			(effects
-				(font
-					(size 1.27 1.27)
-				)
-				(hide yes)
-			)
-		)
-		(property "Description" "Generic connector, single row, 01x24, script generated (kicad-library-utils/schlib/autogen/connector/)"
-			(at 241.3 71.12 0)
-			(effects
-				(font
-					(size 1.27 1.27)
-				)
-				(hide yes)
-			)
-		)
-		(pin "14"
-		)
-		(pin "9"
-		)
-		(pin "13"
-		)
-		(pin "20"
-		)
-		(pin "1"
-		)
-		(pin "23"
-		)
-		(pin "3"
-		)
-		(pin "4"
-		)
-		(pin "10"
-		)
-		(pin "11"
-		)
-		(pin "8"
-		)
-		(pin "5"
-		)
-		(pin "7"
-		)
-		(pin "6"
-		)
-		(pin "2"
-		)
-		(pin "12"
-		)
-		(pin "15"
-		)
-		(pin "16"
-		)
-		(pin "17"
-		)
-		(pin "18"
-		)
-		(pin "19"
-		)
-		(pin "21"
-		)
-		(pin "22"
-		)
-		(pin "24"
-		)
-		(instances
-			(project "Eink-Driver"
-				(path "/ff08cec3-484d-4cc6-8498-b7b3b5dcf0bf"
-					(reference "J3")
-					(unit 1)
-				)
